File: kicad/silakka60mod.kicad_sch (KiCad schematic)
At the start: 63 parts, among them J1 AudioJack4, J2 AudioJack4, U1 RP2040_Zero

Commit message: Add files via upload
Parts:
- removed J2: AudioJack4, Connector_Audio:Jack_3.5mm_PJ320D_Horizontal, symbol Connector_Audio:AudioJack4
- D1, D10, D11, D12, D13, D14, D15, D16, D17, D18, D19, D2, D20, D21, D22, D23, D24, D25, D26, D27, D28, D29, D3, D30, D4, D5, D6, D7, D8, D9: footprint ScottoKeebs_Components:Diode_DO-35 -> SCOTTOKEEBS components:Diode_DO-35
- S1, S10, S11, S12, S13, S14, S15, S16, S17, S18, S19, S2, S20, S21, S22, S23, S24, S25, S26, S27, S28, S29, S3, S30, S4, S5, S6, S7, S8, S9: footprint kbd:CherryMX_MidHeight_Hotswap -> kbd:keyswitch_cherrymx_hotswap_1u
- U1: footprint ScottoKeebs_MCU:RP2040_Zero -> SCOTTOKEEBS mcu:RP2040_Zero

Commit message: Add files via upload
Parts:
- added D31, D32, D33, D34, D35, D36, D37, D38, D39, D40, D41, D42, D43, D44, D45, D46, D47, D48, D49, D50, D51, D52, D53, D54, D55, D56, D57, D58, D59, D60: Diode, SCOTTOKEEBS components:Diode_DO-35, symbol ScottoKeebs:Placeholder_Diode
- added J2: AudioJack4, Connector_Audio:Jack_3.5mm_PJ320D_Horizontal, symbol Connector_Audio:AudioJack4
- added S31, S32, S33, S34, S35, S36, S37, S38, S39, S40, S41, S42, S43, S44, S45, S46, S47, S48, S49, S50, S51, S52, S53, S54, S55, S56, S57, S58, S59, S60: Keyswitch, kbd:keyswitch_cherrymx_hotswap_1u, symbol ScottoKeebs:Placeholder_Keyswitch
- added U2: RP2040_Zero, SCOTTOKEEBS mcu:RP2040_Zero, symbol ScottoKeebs:MCU_RP2040_Zero
Connections:
- new net: D49.2 (A), S49.1
- new net: D46.2 (A), S46.1
- new net: D40.2 (A), S40.1
- new net: D56.2 (A), S56.1
- new net: D39.2 (A), S39.1
- new net: D31.2 (A), S31.1
- new net: D52.2 (A), S52.1
- new net: D58.2 (A), S58.1
- new net: D45.2 (A), S45.1
- new net: D48.2 (A), S48.1
- new net: D44.2 (A), S44.1
- new net: D50.2 (A), S50.1
- new net: D60.2 (A), S60.1
- new net: D37.2 (A), S37.1
- new net: D36.2 (A), S36.1
- new net: D54.2 (A), S54.1
- new net: D43.2 (A), S43.1
- new net: D42.2 (A), S42.1
- new net: D34.2 (A), S34.1
- new net: D51.2 (A), S51.1
- new net: D47.2 (A), S47.1
- new net: D33.2 (A), S33.1
- new net: D55.2 (A), S55.1
- new net: D38.2 (A), S38.1
- new net: D57.2 (A), S57.1
- new net: D59.2 (A), S59.1
- new net: D41.2 (A), S41.1
- new net: D32.2 (A), S32.1
- new net: D53.2 (A), S53.1
- new net: D35.2 (A), S35.1
- new net COL0b: S31.2, S37.2, S43.2, S49.2, S55.2, U2.8 (7)
- new net COL1b: S32.2, S38.2, S44.2, S50.2, S56.2, U2.9 (8)
- new net COL2b: S33.2, S39.2, S45.2, S51.2, S57.2, U2.10 (9)
- new net COL3b: S34.2, S40.2, S46.2, S52.2, S58.2, U2.11 (10)
- new net COL4b: S35.2, S41.2, S47.2, S53.2, S59.2, U2.12 (11)
- new net COL5b: S36.2, S42.2, S48.2, S54.2, S60.2, U2.13 (12)
- new net GNDb: J2.S, U2.22 (GND)
- new net ROW0b: D31.1 (K), D32.1 (K), D33.1 (K), D34.1 (K), D35.1 (K), D36.1 (K), U2.3 (2)
- new net ROW1b: D37.1 (K), D38.1 (K), D39.1 (K), D40.1 (K), D41.1 (K), D42.1 (K), U2.4 (3)
- new net ROW2b: D43.1 (K), D44.1 (K), D45.1 (K), D46.1 (K), D47.1 (K), D48.1 (K), U2.5 (4)
- new net ROW3b: D49.1 (K), D50.1 (K), D51.1 (K), D52.1 (K), D53.1 (K), D54.1 (K), U2.6 (5)
- new net ROW4b: D55.1 (K), D56.1 (K), D57.1 (K), D58.1 (K), D59.1 (K), D60.1 (K), U2.7 (6)
- new net RXb: J2.T, U2.2 (1)
- new net TXb: J2.R1, U2.1 (0)
- new net VCCb: J2.R2, U2.21 (3V3)
Other:
- moved on the sheet: D1, D10, D11, D12, D13, D14, D15, D16, D17, D18, D19, D2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
